Commit message: gazebo_diff_drive

File: description/robot.urdf.xacro (robot description, xacro)
@@ -2,3 +2,4 @@
 <robot xmlns:xacro="http://www.ros.org/wiki/xacro"  name="robot">
     <xacro:include filename="robot_core.xacro"/>
+    <xacro:include filename="gazebo_control.xacro"/>
 </robot>

File: description/robot_core.xacro (robot description, xacro)
@@ -1,4 +1,5 @@
 <?xml version="1.0"?>
-<robot xmlns:xacro="http://www.ros.org/wiki/xacro"  >
+<robot xmlns:xacro="http://www.ros.org/wiki/xacro" >
+    <xacro:include filename="inertial_macros.xacro"/>
     <material name="grey">
         <color rgba="0.7 0.7 0.7 1"/>
@@ -25,5 +26,11 @@
             <origin xyz="0 0 0.1" rpy="0 0 0" />
         </collision>
+        <xacro:inertial_box mass="0.5" x="0.6" y="0.4" z="0.2">
+            <origin xyz="0 0 0.1" rpy="0 0 0"/>
+        </xacro:inertial_box>
     </link>
+    <gazebo reference="base_link">
+        <material>Gazebo/White</material>
+    </gazebo>
     <link name="lidar">
         <visual>
@@ -55,5 +62,11 @@
             <origin xyz="0 0 0" rpy="1.57 0 0"/>
         </collision>
+        <xacro:inertial_cylinder mass="0.1" length="0.05" radius="0.1">
+                <origin xyz="0 0 0" rpy="1.57 0 0"/>
+        </xacro:inertial_cylinder>
     </link>
+    <gazebo reference="left_wheel">
+        <material>Gazebo/Blue</material>
+    </gazebo>
     <link name="right_wheel">
         <visual>
@@ -70,5 +83,11 @@
             <origin xyz="0 0 0" rpy="1.57 0 0" />
         </collision>
+        <xacro:inertial_cylinder mass="0.1" length="0.05" radius="0.1">
+                <origin xyz="0 0 0" rpy="1.57 0 0"/>
+        </xacro:inertial_cylinder>
     </link>
+    <gazebo reference="right_wheel">
+        <material>Gazebo/Blue</material>
+    </gazebo>
     <link name="caster_wheel">
         <visual>
@@ -85,5 +104,13 @@
             <origin xyz="0 0 0" rpy="0 0 0"/>
         </collision>
+        <xacro:inertial_sphere mass="0.1" radius="0.05">
+            <origin xyz="0 0 0" rpy="0 0 0"/>
+        </xacro:inertial_sphere>
     </link>
+    <gazebo reference="caster_wheel">
+        <material>Gazebo/Black</material>
+        <mu1 value="0.001"/>
+        <mu2 value="0.001"/>
+    </gazebo>
     <joint name="base_joint" type="fixed">
         <parent link ="base_footprint" />
@@ -102,5 +129,5 @@
         <axis xyz= "0 1 0" />
     </joint>
-    <joint name="base_right_wheeL_joint" type="continuous">
+    <joint name="base_right_wheel_joint" type="continuous">
         <parent link="base_link" />
         <child link="right_wheel" />

Commit message: Update robot simulation and Nav2 configuration

File: description/robot.urdf.xacro (robot description, xacro)
@@ -2,4 +2,7 @@
 <robot xmlns:xacro="http://www.ros.org/wiki/xacro"  name="robot">
     <xacro:include filename="robot_core.xacro"/>
-    <xacro:include filename="gazebo_control.xacro"/>
+    <!--xacro:include filename="gazebo_control.xacro">/-->
+    <xacro:include filename="ros2_control.xacro"/>
+    <xacro:include filename="lidar.xacro"/>
+    <xacro:include filename="camera.xacro"/>
 </robot>

File: description/robot_core.xacro (robot description, xacro)
@@ -11,6 +11,13 @@
         <color rgba="1 1 1 1"/>
     </material>
-    <link name="base_footprint" />
-    <link name="base_link">
+    <link name="base_link" />
+    <joint name="base_footprint_joint" type="fixed">
+        <parent link="base_link"/>
+        <child link="base_footprint"/>
+        <origin xyz="0 0 0" rpy="0 0 0"/>
+    </joint>
+    <link name="base_footprint">
+    </link>
+    <link name="chassis">
         <visual>
             <geometry>
@@ -30,22 +37,7 @@
         </xacro:inertial_box>
     </link>
-    <gazebo reference="base_link">
+    <gazebo reference="chassis">
         <material>Gazebo/White</material>
     </gazebo>
-    <link name="lidar">
-        <visual>
-            <geometry>
-                <cylinder radius="0.1" length ="0.05" />
-            </geometry>
-            <origin xyz="0 0 0" rpy="0 0 0" />
-            <material name="white" />
-        </visual>
-        <collision>
-            <geometry>
-                <cylinder radius="0.1" length ="0.05" />
-            </geometry>
-            <origin xyz="0 0 0" rpy="0 0 0" />
-        </collision>
-    </link>
     <link name="left_wheel">
         <visual>
@@ -114,15 +106,10 @@
     </gazebo>
     <joint name="base_joint" type="fixed">
-        <parent link ="base_footprint" />
-        <child link="base_link" />
+        <parent link ="base_link" />
+        <child link="chassis" />
         <origin xyz="0 0 0.1" rpy="0 0 0" />
     </joint>
-    <joint name="base_lidar_joint" type="fixed">
-        <parent link="base_link" />
-        <child link="lidar" />
-        <origin xyz="0 0 0.225" rpy="0 0 0" />
-    </joint>
     <joint name="base_left_wheel_joint" type="continuous">
-        <parent link="base_link" />
+        <parent link="chassis" />
         <child link="left_wheel" />
         <origin xyz="-0.15 0.225 0" rpy="0 0 0" />
@@ -130,5 +117,5 @@
     </joint>
     <joint name="base_right_wheel_joint" type="continuous">
-        <parent link="base_link" />
+        <parent link="chassis" />
         <child link="right_wheel" />
         <origin xyz="-0.15 -0.225 0" rpy="0 0 0" />
@@ -136,5 +123,5 @@
     </joint>
     <joint name="base_caster_wheel_joint" type="fixed">
-        <parent link ="base_link"/>
+        <parent link ="chassis"/>
         <child link ="caster_wheel"/>
         <origin xyz="0.2 0 -0.05" rpy="0 0 0"/>
